File: 4LayerV1/ATSAMA5D27-1G.sch (KiCad schematic (older format))
At the start: 172 parts, among them J1 Conn_01x16, J2 Conn_01x12, J3 USB_B_Micro, J4 Conn_01x02, J5 Conn_01x02, J6 1051620001, J7 USB_A_Micro, Q1 BSS138, Q2 BSS138, Q3 BSS138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

Commit message: Adding LCD pins.
Connections:
- net I2C_TWD0: now also U1.M2 (PD29); no longer U1.G7 (PB31)
- net LCDDAT[14]: now reaches U1.A3 (PB25)
- net LCDDAT[9]: now reaches U1.A4 (PB20)
- net LCDDAT[7]: now reaches U1.A5 (PB18)
- net LCDDAT[3]: now reaches U1.A6 (PB14)
- net LCDDAT[0]: now reaches U1.A7 (PB11)
- net PMIC_IRQ_PB10: now reaches U1.A8 (PB10)
- net PMIC_IRQ_PB10: now also R9.2, U2.12 (nIRQ)
- net LCDDAT[12]: now reaches U1.B3 (PB23)
- net LCDDAT[8]: now reaches U1.B4 (PB19)
- net LCDDAT[5]: now reaches U1.B5 (PB16)
- net LCDDAT[1]: now reaches U1.B6 (PB12)
- net LCDDAT[11]: now reaches U1.C3 (PB22)
- net LCDDAT[6]: now reaches U1.C4 (PB17)
- net LCDDAT[17]: now reaches U1.D2 (PB28)
- net LCDDAT[10]: now reaches U1.D3 (PB21)
- net LCDDAT[13]: now reaches U1.E2 (PB24)
- net LCDDAT[4]: now reaches U1.E4 (PB15)
- net LCDDAT[16]: now reaches U1.F4 (PB27)
- net LCDDAT[15]: now reaches U1.G3 (PB26)
- net LCDHSYNC: now reaches U1.L11 (PC6)
- net LCDVSYNC: now reaches U1.M16 (PC5)
- removed net PMIC_IRQ_PB13: R9.2, U1.C5 (PB13), U2.12 (nIRQ)
- new net LCDDAT[2]: U1.C5 (PB13)
Changed lines of the file:
@@
 Wire Wire Line
 	14600 14100 14350 14100
-Text GLabel 16050 7750 2    39   Input ~ 0
-PMIC_IRQ_PB13
-Wire Wire Line
-	16050 7750 15850 7750
+Text GLabel 16050 7450 2    39   Input ~ 0
+PMIC_IRQ_PB10
 Text GLabel 3800 8550 0    39   Input ~ 0
-PMIC_IRQ_PB13
+PMIC_IRQ_PB10
 Text GLabel 14500 7650 2    39   Input ~ 0
 PMIC_CHGLEV_PA12
@@
 Text GLabel 19350 9550 2    39   Input ~ 0
 ADTRG-IRQ
-Wire Wire Line
-	16050 9550 15850 9550
 Text GLabel 17700 6450 2    39   Input ~ 0
 I2C_TWCK0
 Wire Wire Line
 	17700 6450 17500 6450
-Text GLabel 16050 9550 2    39   Input ~ 0
+Text GLabel 19360 9350 2    39   Input ~ 0
 I2C_TWD0
 Text GLabel 13000 14100 0    39   Input ~ 0
@@
 NoConn ~ 2650 1850
 NoConn ~ 3800 15700
+Text GLabel 16050 7550 2    39   Input ~ 0
+LCDDAT[0]
+Text GLabel 16050 7650 2    39   Input ~ 0
+LCDDAT[1]
+Text GLabel 16050 7750 2    39   Input ~ 0
+LCDDAT[2]
+Text GLabel 16050 7850 2    39   Input ~ 0
+LCDDAT[3]
+Text GLabel 16050 7950 2    39   Input ~ 0
+LCDDAT[4]
+Text GLabel 16050 8050 2    39   Input ~ 0
+LCDDAT[5]
+Text GLabel 16050 8150 2    39   Input ~ 0
+LCDDAT[6]
+Text GLabel 16050 8250 2    39   Input ~ 0
+LCDDAT[7]
+Text GLabel 16050 8350 2    39   Input ~ 0
+LCDDAT[8]
+Text GLabel 16050 8450 2    39   Input ~ 0
+LCDDAT[9]
+Text GLabel 16050 8550 2    39   Input ~ 0
+LCDDAT[10]
+Text GLabel 16050 8650 2    39   Input ~ 0
+LCDDAT[11]
+Text GLabel 16050 8750 2    39   Input ~ 0
+LCDDAT[12]
+Text GLabel 16050 8850 2    39   Input ~ 0
+LCDDAT[13]
+Text GLabel 16050 8950 2    39   Input ~ 0
+LCDDAT[14]
+Text GLabel 16050 9050 2    39   Input ~ 0
+LCDDAT[15]
+Text GLabel 16050 9150 2    39   Input ~ 0
+LCDDAT[16]
+Text GLabel 16050 9250 2    39   Input ~ 0
+LCDDAT[17]
+Wire Wire Line
+	19360 9350 19100 9350
+Text GLabel 17700 6950 2    39   Input ~ 0
+LCDVSYNC
+Text GLabel 17700 7050 2    39   Input ~ 0
+LCDHSYNC
+Wire Wire Line
+	17700 7050 17500 7050
+Wire Wire Line
+	17700 6950 17500 6950
+Wire Wire Line
+	15850 7550 16050 7550
+Wire Wire Line
+	15850 7650 16050 7650
+Wire Wire Line
+	15850 7750 16050 7750
+Wire Wire Line
+	15850 7850 16050 7850
+Wire Wire Line
+	16050 7950 15850 7950
+Wire Wire Line
+	15850 8050 16050 8050
+Wire Wire Line
+	16050 8150 15850 8150
+Wire Wire Line
+	15850 8250 16050 8250
+Wire Wire Line
+	16050 8350 15850 8350
+Wire Wire Line
+	15850 8450 16050 8450
+Wire Wire Line
+	16050 8550 15850 8550
+Wire Wire Line
+	15850 8650 16050 8650
+Wire Wire Line
+	16050 8750 15850 8750
+Wire Wire Line
+	15850 8850 16050 8850
+Wire Wire Line
+	16050 8950 15850 8950
+Wire Wire Line
+	15850 9050 16050 9050
+Wire Wire Line
+	16050 9150 15850 9150
+Wire Wire Line
+	15850 9250 16050 9250
+Wire Wire Line
+	16050 7450 15850 7450
 $EndSCHEMATC
