File: 4LayerV1/ATSAMA5D27-1G.sch (KiCad schematic (older format))
At the start: 172 parts, among them J1 Conn_01x16, J2 Conn_01x12, J3 USB_B_Micro, J4 Conn_01x02, J5 Conn_01x02, J6 1051620001, J7 USB_B_Micro, Q1 BSS138, Q2 BSS138, Q3 BSS138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

Commit message: Swap USB micro-B for USB micro-A in schematic.
This indicates that the lower USB port is a USB Host interface that
supplies 5V power, as opposed to a USB Device interface that receives 5V
power.
Parts:
- J7: value USB_B_Micro -> USB_A_Micro; symbol Connector:USB_B_Micro -> Connector:USB_A
Connections:
- net CGND: now also J7.5 (Shield); no longer J7.6 (Shield)
- net GND: now also J7.4 (GND); no longer J7.5 (GND)
- no-connect marks 1 -> 2
Changed lines of the file:
@@
 	7500 7700 7600 7700
 $Comp
-L Connector:USB_B_Micro J7
+L Connector:USB_A J7
 U 1 1 5C0AF1F1
 P 4750 15500
 F 0 "J7" V 4759 15829 50  0000 L CNN
-F 1 "USB_B_Micro" V 4850 15829 50  0000 L CNN
+F 1 "USB_A_Micro" V 4850 15829 50  0000 L CNN
 F 2 "10104111-0001LF:FRAMATOME_10104111-0001LF" H 4900 15450 50  0001 C CNN
 F 3 "https://cdn.amphenol-icc.com/media/wysiwyg/files/drawing/10104111.pdf" H 4900 15450 50  0001 C CNN
@@
 SWDIO
 NoConn ~ 2650 1850
+NoConn ~ 3800 15700
 $EndSCHEMATC

Commit message: Create local footprint library and copy over custom footprints.
In theory you should be able to update the PCB from the Schematic now
with no changes, however, there seems to be an issue with the USB
port PCB layout not matching the schematic - perhaps due to the swap
from a USB B to a USB A component?
Parts:
- J3: footprint OSD3358-CHIP:USB_Micro-B_Molex-105017-0001 -> ATSAMA5D27-1G:USB_Micro-B_Molex-105017-0001
- J6: footprint 1051620001:1051620001 -> ATSAMA5D27-1G:1051620001
- J7: footprint 10104111-0001LF:FRAMATOME_10104111-0001LF -> ATSAMA5D27-1G:FRAMATOME_10104111-0001LF
- L11, L12, L6: footprint footprints:L_0603 -> ATSAMA5D27-1G:L_0603
- NT1, NT2: footprint footprints:NetTie-2_SMD_Padsmall -> ATSAMA5D27-1G:NetTie-2_SMD_Padsmall
- PB1: footprint OSD3358-CHIP:MINI_PUSHBUTTON -> ATSAMA5D27-1G:MINI_PUSHBUTTON
Changed lines of the file:
@@
 F 0 "J3" V 3509 15829 50  0000 L CNN
 F 1 "USB_B_Micro" V 3600 15829 50  0000 L CNN
-F 2 "OSD3358-CHIP:USB_Micro-B_Molex-105017-0001" H 3650 15450 50  0001 C CNN
+F 2 "ATSAMA5D27-1G:USB_Micro-B_Molex-105017-0001" H 3650 15450 50  0001 C CNN
 F 3 "~" H 3650 15450 50  0001 C CNN
 F 4 "Molex" H 3500 15500 50  0001 C CNN "Manufacturer_Name"
@@
 F 0 "PB1" V 5042 10297 45  0000 R CNN
 F 1 "POWER-ON" V 4300 10600 45  0000 R CNN
-F 2 "OSD3358-CHIP:MINI_PUSHBUTTON" H 5030 10600 20  0001 C CNN
+F 2 "ATSAMA5D27-1G:MINI_PUSHBUTTON" H 5030 10600 20  0001 C CNN
 F 3 "" H 5000 10450 60  0001 C CNN
 F 4 "C&K" H 5000 10400 50  0001 C CNN "Manufacturer_Name"
@@
 F 0 "L6" V 5150 4400 50  0000 C CNN
 F 1 "MLZ1608N100L" V 5050 4250 50  0000 C CNN
-F 2 "footprints:L_0603" H 5100 4400 50  0001 C CNN
+F 2 "ATSAMA5D27-1G:L_0603" H 5100 4400 50  0001 C CNN
 F 3 "~" H 5100 4400 50  0001 C CNN
 F 4 "TDK" H 5100 4400 50  0001 C CNN "Manufacturer_Name"
@@
 F 0 "L11" V 2600 3800 50  0000 C CNN
 F 1 "MLZ1608N100L" V 2500 3650 50  0000 C CNN
-F 2 "footprints:L_0603" H 2550 3800 50  0001 C CNN
+F 2 "ATSAMA5D27-1G:L_0603" H 2550 3800 50  0001 C CNN
 F 3 "~" H 2550 3800 50  0001 C CNN
 F 4 "TDK" H 2550 3800 50  0001 C CNN "Manufacturer_Name"
@@
 F 0 "L12" V 2600 4750 50  0000 C CNN
 F 1 "MLZ1608N100L" V 2500 4600 50  0000 C CNN
-F 2 "footprints:L_0603" H 2550 4750 50  0001 C CNN
+F 2 "ATSAMA5D27-1G:L_0603" H 2550 4750 50  0001 C CNN
 F 3 "~" H 2550 4750 50  0001 C CNN
 F 4 "TDK" H 2550 4750 50  0001 C CNN "Manufacturer_Name"
@@
 F 0 "J6" H 8300 14065 50  0000 C CNN
 F 1 "1051620001" H 8300 13974 50  0000 C CNN
-F 2 "1051620001:1051620001" H 8800 13900 50  0001 L CNN
+F 2 "ATSAMA5D27-1G:1051620001" H 8800 13900 50  0001 L CNN
 F 3 "https://www.molex.com/pdm_docs/sd/1051620001_sd.pdf" H 8800 13800 50  0001 L CNN
 F 4 "1.45H MICRO SD HEADER WITH D/C P" H 8800 13700 50  0001 L CNN "Description"
@@
 F 0 "J7" V 4759 15829 50  0000 L CNN
 F 1 "USB_A_Micro" V 4850 15829 50  0000 L CNN
-F 2 "10104111-0001LF:FRAMATOME_10104111-0001LF" H 4900 15450 50  0001 C CNN
+F 2 "ATSAMA5D27-1G:FRAMATOME_10104111-0001LF" H 4900 15450 50  0001 C CNN
 F 3 "https://cdn.amphenol-icc.com/media/wysiwyg/files/drawing/10104111.pdf" H 4900 15450 50  0001 C CNN
 F 4 "Amphenol" H 4750 15500 50  0001 C CNN "Manufacturer_Name"
@@
 F 0 "NT1" V 18754 3241 50  0000 L CNN
 F 1 "Net-Tie_2" V 18845 3241 50  0000 L CNN
-F 2 "footprints:NetTie-2_SMD_Padsmall" H 18800 3200 50  0001 C CNN
+F 2 "ATSAMA5D27-1G:NetTie-2_SMD_Padsmall" H 18800 3200 50  0001 C CNN
 F 3 "~" H 18800 3200 50  0001 C CNN
 	1    18800 3200
@@
 F 0 "NT2" V 16454 3941 50  0000 L CNN
 F 1 "Net-Tie_2" V 16545 3941 50  0000 L CNN
-F 2 "footprints:NetTie-2_SMD_Padsmall" H 16500 3900 50  0001 C CNN
+F 2 "ATSAMA5D27-1G:NetTie-2_SMD_Padsmall" H 16500 3900 50  0001 C CNN
 F 3 "~" H 16500 3900 50  0001 C CNN
 	1    16500 3900

Commit message: Squeezing in a 0R on the USB A power pin.
Parts:
- added R13: 0R, Resistor_SMD:R_0402_1005Metric, symbol Device:R_Small
- J7: value USB_A_Micro -> USB_AB_Micro; symbol Connector:USB_A -> Connector:USB_OTG
Connections:
- net CGND: now also J7.6 (Shield); no longer J7.5 (Shield)
- net GND: now also J7.5 (GND); no longer J7.4 (GND)
- net VBUS: now also R13.1; no longer J7.1 (VBUS)
- net USBA_M renamed USBA_N
- net USBB_M renamed USBB_N
- new net: J7.1 (VBUS), R13.2
- no-connect marks 2 -> 3
Other:
- note added: "Fit R13 if J7 is used\nas USB Host. Remove\nR13 if J7 is used as\nUSB Device"
Changed lines of the file:
@@
 USBA_P
 Text GLabel 3950 15600 2    39   Input ~ 0
-USBA_M
+USBA_N
 Wire Wire Line
 	18250 2000 17850 2000
@@
 USBA_P
 Text GLabel 18250 2100 2    39   Input ~ 0
-USBA_M
+USBA_N
 Text GLabel 1250 2600 0    39   Input ~ 0
 VDD_3V3
 Text GLabel 18250 2350 2    39   Input ~ 0
-USBB_M
+USBB_N
 Text GLabel 18250 2250 2    39   Input ~ 0
 USBB_P
@@
 $EndComp
 Text GLabel 4750 14400 0    39   Input ~ 0
-USBB_M
+USBB_N
 Text GLabel 4750 14500 0    39   Input ~ 0
 USBB_P
@@
 	7500 7700 7600 7700
 $Comp
-L Connector:USB_A J7
+L Connector:USB_OTG J7
 U 1 1 5C0AF1F1
 P 4750 15500
 F 0 "J7" V 4759 15829 50  0000 L CNN
-F 1 "USB_A_Micro" V 4850 15829 50  0000 L CNN
+F 1 "USB_AB_Micro" V 4850 15829 50  0000 L CNN
 F 2 "ATSAMA5D27-1G:FRAMATOME_10104111-0001LF" H 4900 15450 50  0001 C CNN
 F 3 "https://cdn.amphenol-icc.com/media/wysiwyg/files/drawing/10104111.pdf" H 4900 15450 50  0001 C CNN
@@
 $EndComp
 Text GLabel 5200 15600 2    39   Input ~ 0
-USBB_M
+USBB_N
 Text GLabel 5200 15500 2    39   Input ~ 0
 USBB_P
@@
 	1    0    0    -1
 $EndComp
-Text GLabel 5250 15300 2    39   Input ~ 0
+Text GLabel 5370 15300 2    39   Input ~ 0
 VBUS
-Wire Wire Line
-	5250 15300 5050 15300
 $Comp
 L Device:R_Small R14
@@
 F 3 "" H 6550 15150 50  0001 C CNN
 	1    6550 15150
-	0    1    1    0
-$EndComp
-$Comp
-L Device:R_Small R36
-U 1 1 5C307E80
-P 6750 15150
-F 0 "R36" V 6850 15150 50  0000 C CNN
-F 1 "0R" V 6650 15150 50  0000 C CNN
-F 2 "Resistor_SMD:R_0402_1005Metric" H 6750 15150 50  0001 C CNN
-F 3 "~" H 6750 15150 50  0001 C CNN
-F 4 "Stackpole" H 6750 15150 50  0001 C CNN "Manufacturer_Name"
-F 5 "RMCF0402ZT0R00" H 6750 15150 50  0001 C CNN "Manufacturer_Part_Number"
-	1    6750 15150
 	0    1    1    0
 $EndComp
@@
 NoConn ~ 2650 1850
 NoConn ~ 3800 15700
+NoConn ~ 5050 15700
+Wire Wire Line
+	5050 15300 5110 15300
+Text Notes 4910 16270 0    50   ~ 0
+Fit R13 if J7 is used\nas USB Host. Remove\nR13 if J7 is used as\nUSB Device
+Wire Wire Line
+	5370 15300 5310 15300
+$Comp
+L Device:R_Small R36
+U 1 1 5C307E80
+P 6750 15150
+F 0 "R36" V 6850 15150 50  0000 C CNN
+F 1 "0R" V 6650 15150 50  0000 C CNN
+F 2 "Resistor_SMD:R_0402_1005Metric" H 6750 15150 50  0001 C CNN
+F 3 "~" H 6750 15150 50  0001 C CNN
+F 4 "Stackpole" H 6750 15150 50  0001 C CNN "Manufacturer_Name"
+F 5 "RMCF0402ZT0R00" H 6750 15150 50  0001 C CNN "Manufacturer_Part_Number"
+	1    6750 15150
+	0    1    1    0
+$EndComp
+$Comp
+L Device:R_Small R13
+U 1 1 64311672
+P 5210 15300
+F 0 "R13" V 5310 15300 50  0000 C CNN
+F 1 "0R" V 5110 15300 50  0000 C CNN
+F 2 "Resistor_SMD:R_0402_1005Metric" H 5210 15300 50  0001 C CNN
+F 3 "~" H 5210 15300 50  0001 C CNN
+F 4 "Stackpole" H 5210 15300 50  0001 C CNN "Manufacturer_Name"
+F 5 "RMCF0402ZT0R00" H 5210 15300 50  0001 C CNN "Manufacturer_Part_Number"
+	1    5210 15300
+	0    1    1    0
+$EndComp
 $EndSCHEMATC
